File: RAM.sch (KiCad schematic (older format))
At the start: 6 parts

Commit message: Much progress
Changed lines of the file:
@@
 $Descr A4 11693 8268
 encoding utf-8
-Sheet 5 7
+Sheet 6 7
 Title ""
 Date ""
@@
 $EndDescr
 Text HLabel 2700 2750 0    50   Input ~ 0
-RA[12..0]
+RA[11..0]
 Wire Bus Line
 	2750 2750 2700 2750
