File: ROM.sch (KiCad schematic (older format))
At the start: 2 parts

Commit message: idk
Connections:
- net FU~CS~ is gone; now on net ~CS~: U?.22 (~CS~)
- net RD0: now also U?.13 (D0); no longer U?.18 (D4)
- net RD1: now also U?.14 (D1); no longer U?.17 (D3)
- net RD10: now also U?.15 (D2); no longer U?.19 (D5)
- net RD11: now also U?.17 (D3); no longer U?.15 (D2)
- net RD12: now also U?.18 (D4); no longer U?.20 (D6)
- net RD13: now also U?.19 (D5); no longer U?.14 (D1)
- net RD14: now also U?.20 (D6); no longer U?.21 (D7)
- net RD15: now also U?.21 (D7); no longer U?.13 (D0)
- net RD2: now also U?.15 (D2); no longer U?.19 (D5)
- net RD3: now also U?.17 (D3); no longer U?.15 (D2)
- net RD4: now also U?.18 (D4); no longer U?.20 (D6)
- net RD5: now also U?.19 (D5); no longer U?.14 (D1)
- net RD6: now also U?.20 (D6); no longer U?.21 (D7)
- net RD7: now also U?.21 (D7); no longer U?.13 (D0)
- net RD8: now also U?.13 (D0); no longer U?.18 (D4)
- net RD9: now also U?.14 (D1); no longer U?.17 (D3)
- net FL~CS~ renamed ~CS~
- net R~W~ renamed L~WE~
- net L~WE~: no longer U?.31 (~WE~)
- net ~R~W renamed ~OE~
- new net U~WE~: U?.31 (~WE~)
Changed lines of the file:
@@
 $Descr A4 11693 8268
 encoding utf-8
-Sheet 6 7
+Sheet 4 7
 Title ""
 Date ""
@@
 $EndComp
 Text HLabel 3450 3400 2    50   Input ~ 0
-~R~W
+~OE~
 Text HLabel 3450 3200 2    50   Input ~ 0
-FL~CS~
+~CS~
 Entry Wire Line
 	2350 4300 2450 4200
@@
 RA2
 $Comp
+L power:GND #PWR?
+U 1 1 60E1A140
+P 3450 5900
+AR Path="/5F723900/60E1A140" Ref="#PWR?"  Part="1"
+AR Path="/60D70CB4/60E1A140" Ref="#PWR?"  Part="1"
+F 0 "#PWR?" H 3450 5650 50  0001 C CNN
+F 1 "GND" H 3450 5750 50  0000 C CNN
+F 2 "" H 3450 5900 50  0001 C CNN
+F 3 "" H 3450 5900 50  0001 C CNN
+	1    3450 5900
+	1    0    0    -1
+$EndComp
+Text Label 3450 2100 0    50   ~ 0
+RD0
+Text Label 3450 2200 0    50   ~ 0
+RD1
+Text Label 3450 2300 0    50   ~ 0
+RD2
+Text Label 3450 2400 0    50   ~ 0
+RD3
+Text Label 3450 2500 0    50   ~ 0
+RD4
+Text Label 3450 2600 0    50   ~ 0
+RD5
+Text Label 3450 2700 0    50   ~ 0
+RD6
+Text Label 3450 2800 0    50   ~ 0
+RD7
+Entry Wire Line
+	3750 2100 3650 2200
+Entry Wire Line
+	3750 2000 3650 2100
+Entry Wire Line
+	3750 2300 3650 2400
+Entry Wire Line
+	3750 2200 3650 2300
+Entry Wire Line
+	3750 2500 3650 2600
+Entry Wire Line
+	3750 2400 3650 2500
+Entry Wire Line
+	3750 2700 3650 2800
+Entry Wire Line
+	3750 2600 3650 2700
+Wire Wire Line
+	3450 2700 3650 2700
+Wire Wire Line
+	3450 2500 3650 2500
+Wire Wire Line
+	3450 2300 3650 2300
+Wire Wire Line
+	3450 2100 3650 2100
+Wire Wire Line
+	3450 2200 3650 2200
+Wire Wire Line
+	3450 2400 3650 2400
+Wire Wire Line
+	3450 2600 3650 2600
+Wire Wire Line
+	3450 2800 3650 2800
+Wire Wire Line
+	2650 5900 2450 5900
+Wire Wire Line
+	2650 5800 2450 5800
+Entry Wire Line
+	2350 5900 2450 5800
+Wire Wire Line
+	2650 5700 2450 5700
+Entry Wire Line
+	2350 5800 2450 5700
+Entry Wire Line
+	2350 6000 2450 5900
+Text Label 2650 5700 2    50   ~ 0
+RA17
+Text Label 2650 5800 2    50   ~ 0
+RA18
+Text Label 2650 5900 2    50   ~ 0
+RA19
+Wire Wire Line
+	2650 3700 2450 3700
+Wire Wire Line
+	2650 3600 2450 3600
+Entry Wire Line
+	2350 3700 2450 3600
+Wire Wire Line
+	2650 3500 2450 3500
+Entry Wire Line
+	2350 3600 2450 3500
+Entry Wire Line
+	2350 3800 2450 3700
+Text Label 2650 3500 2    50   ~ 0
+RA17
+Text Label 2650 3600 2    50   ~ 0
+RA18
+Text Label 2650 3700 2    50   ~ 0
+RA19
+Text HLabel 3450 3300 2    50   Input ~ 0
+L~WE~
+Wire Bus Line
+	2300 1600 3750 1600
+Wire Bus Line
+	2350 2000 2300 2000
+Text HLabel 2300 1600 0    50   BiDi ~ 0
+D[15..0]
+Text HLabel 2300 2000 0    50   Input ~ 0
+A[23..1]
+Text Label 3450 5000 0    50   ~ 0
+RD15
+Text Label 3450 4900 0    50   ~ 0
+RD14
+Text Label 3450 4800 0    50   ~ 0
+RD13
+Text Label 3450 4700 0    50   ~ 0
+RD12
+Text Label 3450 4600 0    50   ~ 0
+RD11
+Text Label 3450 4500 0    50   ~ 0
+RD10
+Text Label 3450 4400 0    50   ~ 0
+RD9
+Text Label 3450 4300 0    50   ~ 0
+RD8
+Wire Wire Line
+	3450 4900 3650 4900
+Wire Wire Line
+	3450 4700 3650 4700
+Wire Wire Line
+	3450 4500 3650 4500
+Wire Wire Line
+	3450 4300 3650 4300
+Wire Wire Line
+	3450 4400 3650 4400
+Wire Wire Line
+	3450 4600 3650 4600
+Wire Wire Line
+	3450 4800 3650 4800
+Wire Wire Line
+	3450 5000 3650 5000
+Entry Wire Line
+	3750 4300 3650 4400
+Entry Wire Line
+	3750 4200 3650 4300
+Entry Wire Line
+	3750 4500 3650 4600
+Entry Wire Line
+	3750 4400 3650 4500
+Entry Wire Line
+	3750 4700 3650 4800
+Entry Wire Line
+	3750 4600 3650 4700
+Entry Wire Line
+	3750 4900 3650 5000
+Entry Wire Line
+	3750 4800 3650 4900
+Text HLabel 3450 5500 2    50   Input ~ 0
+U~WE~
+Text HLabel 3450 5400 2    50   Input ~ 0
+~CS~
+Text HLabel 3450 5600 2    50   Input ~ 0
+~OE~
+$Comp
 L GW_RAM:Flash-512Kx8-PLCC-32 U?
 U 1 1 60E1A13A
@@
 	1    0    0    -1
 $EndComp
-$Comp
-L power:GND #PWR?
-U 1 1 60E1A140
-P 3450 5900
-AR Path="/5F723900/60E1A140" Ref="#PWR?"  Part="1"
-AR Path="/60D70CB4/60E1A140" Ref="#PWR?"  Part="1"
-F 0 "#PWR?" H 3450 5650 50  0001 C CNN
-F 1 "GND" H 3450 5750 50  0000 C CNN
-F 2 "" H 3450 5900 50  0001 C CNN
-F 3 "" H 3450 5900 50  0001 C CNN
-	1    3450 5900
-	1    0    0    -1
-$EndComp
-Text HLabel 3450 5600 2    50   Input ~ 0
-~R~W
-Text HLabel 3450 5400 2    50   Input ~ 0
-FU~CS~
-Text Label 3450 2500 0    50   ~ 0
-RD0
-Text Label 3450 2400 0    50   ~ 0
-RD1
-Text Label 3450 2600 0    50   ~ 0
-RD2
-Text Label 3450 2300 0    50   ~ 0
-RD3
-Text Label 3450 2700 0    50   ~ 0
-RD4
-Text Label 3450 2200 0    50   ~ 0
-RD5
-Text Label 3450 2800 0    50   ~ 0
-RD6
-Text Label 3450 2100 0    50   ~ 0
-RD7
-Text Label 3450 4300 0    50   ~ 0
-RD15
-Text Label 3450 5000 0    50   ~ 0
-RD14
-Text Label 3450 4400 0    50   ~ 0
-RD13
-Text Label 3450 4900 0    50   ~ 0
-RD12
-Text Label 3450 4500 0    50   ~ 0
-RD11
-Text Label 3450 4800 0    50   ~ 0
-RD10
-Text Label 3450 4600 0    50   ~ 0
-RD9
-Text Label 3450 4700 0    50   ~ 0
-RD8
-Wire Wire Line
-	3450 5000 3650 5000
-Wire Wire Line
-	3450 4900 3650 4900
-Entry Wire Line
-	3750 2100 3650 2200
-Entry Wire Line
-	3750 2000 3650 2100
-Wire Wire Line
-	3450 4800 3650 4800
-Wire Wire Line
-	3450 4700 3650 4700
-Entry Wire Line
-	3750 2300 3650 2400
-Entry Wire Line
-	3750 2200 3650 2300
-Wire Wire Line
-	3450 4600 3650 4600
-Wire Wire Line
-	3450 4500 3650 4500
-Entry Wire Line
-	3750 2500 3650 2600
-Entry Wire Line
-	3750 2400 3650 2500
-Wire Wire Line
-	3450 4400 3650 4400
-Wire Wire Line
-	3450 4300 3650 4300
-Entry Wire Line
-	3750 2700 3650 2800
-Entry Wire Line
-	3750 2600 3650 2700
-Wire Wire Line
-	3450 2800 3650 2800
-Wire Wire Line
-	3450 2700 3650 2700
-Entry Wire Line
-	3750 4300 3650 4400
-Entry Wire Line
-	3750 4200 3650 4300
-Wire Wire Line
-	3450 2600 3650 2600
-Wire Wire Line
-	3450 2500 3650 2500
-Entry Wire Line
-	3750 4500 3650 4600
-Entry Wire Line
-	3750 4400 3650 4500
-Wire Wire Line
-	3450 2400 3650 2400
-Wire Wire Line
-	3450 2300 3650 2300
-Entry Wire Line
-	3750 4700 3650 4800
-Entry Wire Line
-	3750 4600 3650 4700
-Wire Wire Line
-	3450 2200 3650 2200
-Wire Wire Line
-	3450 2100 3650 2100
-Entry Wire Line
-	3750 4900 3650 5000
-Entry Wire Line
-	3750 4800 3650 4900
-Wire Wire Line
-	2650 5900 2450 5900
-Wire Wire Line
-	2650 5800 2450 5800
-Entry Wire Line
-	2350 5900 2450 5800
-Wire Wire Line
-	2650 5700 2450 5700
-Entry Wire Line
-	2350 5800 2450 5700
-Entry Wire Line
-	2350 6000 2450 5900
-Text Label 2650 5700 2    50   ~ 0
-RA17
-Text Label 2650 5800 2    50   ~ 0
-RA18
-Text Label 2650 5900 2    50   ~ 0
-RA19
-Wire Wire Line
-	2650 3700 2450 3700
-Wire Wire Line
-	2650 3600 2450 3600
-Entry Wire Line
-	2350 3700 2450 3600
-Wire Wire Line
-	2650 3500 2450 3500
-Entry Wire Line
-	2350 3600 2450 3500
-Entry Wire Line
-	2350 3800 2450 3700
-Text Label 2650 3500 2    50   ~ 0
-RA17
-Text Label 2650 3600 2    50   ~ 0
-RA18
-Text Label 2650 3700 2    50   ~ 0
-RA19
-Text HLabel 3450 5500 2    50   Input ~ 0
-R~W~
-Text HLabel 3450 3300 2    50   Input ~ 0
-R~W~
-Wire Bus Line
-	2300 1600 3750 1600
-Wire Bus Line
-	2350 2000 2300 2000
-Text HLabel 2300 1600 0    50   BiDi ~ 0
-D[15..0]
-Text HLabel 2300 2000 0    50   Input ~ 0
-A[23..1]
 Wire Bus Line
 	3750 1600 3750 4900

Commit message: Much progress
Parts:
- added C? (x2): 2u2, stdpads:C_0603, symbol Device:C_Small
Connections:
- net GND: now also C?.2, C?.2
- net RA1 renamed A1
- net RA10 renamed A10
- net RA11 renamed A11
- net RA12 renamed A12
- net RA13 renamed A13
- net RA14 renamed A14
- net RA15 renamed A15
- net RA16 renamed A16
- net RA17 renamed A17
- net RA18 renamed A18
- net RA19 renamed A19
- net RA2 renamed A2
- net RA3 renamed A3
- net RA4 renamed A4
- net RA5 renamed A5
- net RA6 renamed A6
- net RA7 renamed A7
- net RA8 renamed A8
- net RA9 renamed A9
- net RD0 renamed D0
- net RD1 renamed D1
- net RD10 renamed D10
- net RD11 renamed D11
- net RD12 renamed D12
- net RD13 renamed D13
- net RD14 renamed D14
- net RD15 renamed D15
- net RD2 renamed D2
- net RD3 renamed D3
- net RD4 renamed D4
- net RD5 renamed D5
- net RD6 renamed D6
- net RD7 renamed D7
- net RD8 renamed D8
- net RD9 renamed D9
- new net +5V: C?.1, C?.1
