File: Control.sch (KiCad schematic (older format))
At the start: 1 part, among them U1 XC95144XL-TQ100

Commit message: idk
Connections:
- net A14 is gone; now on net RU~CS~: U1.86 (P86)
- net A15 is gone; now on net RL~CS~: U1.85 (P85)
- net A18 is gone; now on net Acc~BERR~: U1.80 (P80)
- net A19 is gone; now on net Acc~DTACK: U1.79 (P79)
- net A20 is gone; now on net Acc~UDS~: U1.78 (P78)
- net A21 is gone; now on net Acc~LDS~: U1.77 (P77)
- net A23 is gone; now on net Acc~AS~: U1.74 (P74)
- net R~W~ is gone; now on net MacR~W~: U1.34 (P34)
- net Acc~AS~: no longer U1.63 (P63)
- net Acc~BERR~: no longer U1.59 (P59)
- net Acc~DTACK: no longer U1.58 (P58)
- net Acc~LDS~: no longer U1.61 (P61)
- net Acc~UDS~: no longer U1.60 (P60)
- net Mac~LDS~: no longer U1.95 (P95)
- net Mac~UDS~: no longer U1.96 (P96)
- net RL~CS~: no longer U1.64 (P64)
- net RU~CS~: no longer U1.65 (P65)
- net MacA23: now reaches U1.11 (P11)
- net MacA22: now reaches U1.12 (P12)
- net MacA21: now reaches U1.13 (P13)
- net MacA20: now reaches U1.14 (P14)
- net MacA19: now reaches U1.15 (P15)
- net MacA18: now reaches U1.16 (P16)
- net MacA17: now reaches U1.17 (P17)
- net MacR~W~: now reaches U1.18 (P18)
- net MacA~LE~: now reaches U1.2 (I/O/GTS4)
- net MacA~OE~: now reaches U1.3 (I/O/GTS1)
- net AccA23: now reaches U1.35 (P35)
- net AccA22: now reaches U1.36 (P36)
- net AccA21: now reaches U1.37 (P37)
- net AccA20: now reaches U1.39 (P39)
- net MacD~LE~: now reaches U1.4 (I/O/GTS2)
- net AccA19: now reaches U1.40 (P40)
- net AccA18: now reaches U1.41 (P41)
- net AccA17: now reaches U1.42 (P42)
- net AccA16: now reaches U1.43 (P43)
- net AccR~W~: now reaches U1.46 (P46)
- net ~OE~: now reaches U1.54 (P54)
- net RAM01~CS~: now reaches U1.55 (P55)
- net RAM23~CS~: now reaches U1.56 (P56)
- net MacD~OE~: now reaches U1.6 (P6)
- net AccD~LE~: now reaches U1.7 (P7)
- net AccD~OE~: now reaches U1.8 (P8)
- net A11 renamed ~R~W
- net A12 renamed RAM~CS~
- net A13 renamed ROM~CS~
- net A16 renamed AccE
- net A17 renamed Acc~VPA~
- net A22 renamed Acc~VMA~
- net FL~CS~: no longer names the net of U1.68 (P68)
- net FU~CS~: no longer names the net of U1.70 (P70)
- net RDdir: no longer names the net of U1.67 (P67)
- net ~R~W3: no longer names the net of U1.33 (P33)
- new net L~WE~: U1.58 (P58)
- new net RAML~CS~: U1.60 (P60)
- new net RAMU~CS~: U1.61 (P61)
- new net U~WE~: U1.59 (P59)
- new net ~PMCYC~: U1.95 (P95)
Changed lines of the file:
@@
 Text HLabel 3400 5150 0    50   Output ~ 0
 Mac~AS~
-Text HLabel 3400 5350 0    50   Output ~ 0
-Mac~LDS~
-Text HLabel 3400 5450 0    50   Output ~ 0
-Mac~UDS~
 Text HLabel 3400 5250 0    50   Output ~ 0
 Mac~VMA~
 Text HLabel 3400 5550 0    50   Input ~ 0
 Mac~DTACK~
-Text HLabel 3400 5850 0    50   Output ~ 0
-Mac~LDS~
-Text HLabel 3400 5950 0    50   Output ~ 0
-Mac~UDS~
 Text HLabel 3400 5650 0    50   Input ~ 0
 Mac~VPA~
@@
 MacE
 Text HLabel 3400 4950 0    50   Input ~ 0
-R~W~
-Text HLabel 3400 4850 0    50   Input ~ 0
-~R~W3
-Text Label 5400 2950 0    50   ~ 0
-A23
-Text Label 5400 3050 0    50   ~ 0
-A22
-Text Label 5400 3150 0    50   ~ 0
-A21
-Text Label 5400 3250 0    50   ~ 0
-A20
-Text Label 5400 3350 0    50   ~ 0
-A19
-Text Label 5400 3450 0    50   ~ 0
-A18
-Text Label 5400 3550 0    50   ~ 0
-A17
-Text Label 5400 3650 0    50   ~ 0
-A16
-Text Label 5400 3750 0    50   ~ 0
-A15
-Text Label 5400 3850 0    50   ~ 0
-A14
-Text Label 5400 4050 0    50   ~ 0
-A13
-Text Label 5400 4150 0    50   ~ 0
-A12
+MacR~W~
+Text Label 5400 1850 0    50   ~ 0
+AccA22
+Text Label 5400 1950 0    50   ~ 0
+AccA21
+Text Label 5400 2050 0    50   ~ 0
+AccA20
+Text Label 5400 2150 0    50   ~ 0
+AccA19
+Text Label 5400 2250 0    50   ~ 0
+AccA18
+Text Label 5400 2350 0    50   ~ 0
+AccA17
+Text Label 5400 2450 0    50   ~ 0
+AccA16
 Text HLabel 3400 4350 0    50   Input ~ 0
 C8M
 Text HLabel 3400 4050 0    50   Input ~ 0
 C16M
-Text Label 5400 4250 0    50   ~ 0
-A11
+Text HLabel 5400 3350 2    50   Output ~ 0
+Acc~DTACK
+Text HLabel 5400 3450 2    50   Input ~ 0
+Acc~BERR~
+Text HLabel 5400 3250 2    50   Input ~ 0
+Acc~UDS~
+Text HLabel 5400 3150 2    50   Input ~ 0
+Acc~LDS~
+Text HLabel 5400 2950 2    50   Input ~ 0
+Acc~AS~
+Text HLabel 5400 3850 2    50   Output ~ 0
+RU~CS~
+Text HLabel 5400 3750 2    50   Output ~ 0
+RL~CS~
+Text HLabel 5400 4050 2    50   Output ~ 0
+ROM~CS~
+Text HLabel 3400 5450 0    50   Output ~ 0
+Mac~UDS~
+Text HLabel 3400 5350 0    50   Output ~ 0
+Mac~LDS~
+Text HLabel 3400 5850 0    50   Input ~ 0
+~PMCYC~
+Text HLabel 5400 3050 2    50   Input ~ 0
+Acc~VMA~
+Text HLabel 5400 3550 2    50   Input ~ 0
+Acc~VPA~
+Text HLabel 5400 3650 2    50   Input ~ 0
+AccE
+Text Label 5400 1750 0    50   ~ 0
+AccA23
+Text HLabel 5400 2550 2    50   Input ~ 0
+AccR~W~
+Text HLabel 5400 4150 2    50   Output ~ 0
+RAM~CS~
 Text HLabel 5400 4650 2    50   Output ~ 0
-Acc~DTACK
-Text HLabel 5400 4750 2    50   Input ~ 0
-Acc~BERR~
-Text HLabel 5400 4850 2    50   Input ~ 0
-Acc~UDS~
-Text HLabel 5400 4950 2    50   Input ~ 0
-Acc~LDS~
-Text HLabel 5400 5150 2    50   Input ~ 0
-Acc~AS~
-Text HLabel 5400 5350 2    50   Output ~ 0
-RU~CS~
-Text HLabel 5400 5250 2    50   Output ~ 0
-RL~CS~
-Text HLabel 5400 5550 2    50   Output ~ 0
-RDdir
-Text HLabel 5400 5750 2    50   Output ~ 0
-FU~CS~
-Text HLabel 5400 5650 2    50   Output ~ 0
-FL~CS~
+L~WE~
+Text HLabel 5400 4750 2    50   Output ~ 0
+U~WE~
+Text HLabel 5400 4450 2    50   Output ~ 0
+RAM01~CS~
+Text HLabel 5400 4550 2    50   Output ~ 0
+RAM23~CS~
+Text HLabel 5400 4950 2    50   Output ~ 0
+RAMU~CS~
+Text HLabel 5400 4850 2    50   Output ~ 0
+RAML~CS~
+Text HLabel 3400 3350 0    50   Input ~ 0
+MacD~LE~
+Text HLabel 3400 3150 0    50   Input ~ 0
+MacA~LE~
+Text HLabel 3400 3250 0    50   Input ~ 0
+MacA~OE~
+Text HLabel 3400 3450 0    50   Input ~ 0
+MacD~OE~
+Text HLabel 3400 3550 0    50   Input ~ 0
+AccD~LE~
+Text HLabel 3400 3650 0    50   Input ~ 0
+AccD~OE~
+Text HLabel 5400 4250 2    50   Output ~ 0
+~R~W
+Text HLabel 5400 4350 2    50   Output ~ 0
+~OE~
+Text Label 3400 1850 2    50   ~ 0
+MacA22
+Text Label 3400 1950 2    50   ~ 0
+MacA21
+Text Label 3400 2050 2    50   ~ 0
+MacA20
+Text Label 3400 2150 2    50   ~ 0
+MacA19
+Text Label 3400 2250 2    50   ~ 0
+MacA18
+Text Label 3400 2350 2    50   ~ 0
+MacA17
+Text Label 3400 1750 2    50   ~ 0
+MacA23
+Text HLabel 3400 2450 0    50   Output ~ 0
+MacR~W~
 $EndSCHEMATC

Commit message: Much progress
Parts:
- added C26, C27, C28, C29, C30, C31, C32: 2u2, stdpads:C_0603, symbol Device:C_Small
- U1: footprint Package_QFP:TQFP-100_14x14mm_P0.5mm -> stdpads:TQFP-100_14x14mm_P0.5mm
Connections:
- net AccR~W~: no longer U1.46 (P46)
- net Acc~AS~: no longer U1.74 (P74)
- net Acc~BERR~: no longer U1.80 (P80)
- net Acc~DTACK: no longer U1.79 (P79)
- net Acc~LDS~: no longer U1.77 (P77)
- net Acc~UDS~: no longer U1.78 (P78)
- net Acc~VPA~: no longer U1.81 (P81)
- net C16M: no longer U1.23 (I/O/GCK2)
- net C8M: no longer U1.27 (I/O/GCK3)
- net L~WE~: no longer U1.58 (P58)
- net MacE: no longer U1.97 (P97)
- net Mac~AS~: no longer U1.87 (P87)
- net Mac~BERR~: no longer U1.94 (P94)
- net Mac~DTACK~: no longer U1.92 (P92)
- net Mac~LDS~: no longer U1.90 (P90)
- net Mac~UDS~: no longer U1.91 (P91)
- net Mac~VMA~: no longer U1.89 (P89)
- net Mac~VPA~: no longer U1.93 (P93)
- net ROM~CS~: no longer U1.50 (P50)
- net U~WE~: no longer U1.59 (P59)
- net ~OE~: no longer U1.54 (P54)
- net ~RESET~: no longer U1.99 (I/O/GSR)
- net GND: now reaches U1.100 (GND)
- net GND: now also U1.21 (GND), U1.31 (GND), U1.44 (GND), U1.62 (GND), U1.69 (GND), U1.75 (GND), U1.84 (GND), C26.2, C27.2, C28.2, C29.2, C30.2, C31.2, C32.2
- net +3V3: now reaches U1.26 (VCCIO)
- net +3V3: now also U1.38 (VCCIO), U1.5 (VCCINT), U1.51 (VCCIO), U1.57 (VCCINT), U1.88 (VCCIO), U1.98 (VCCINT), C26.1, C27.1, C28.1, C29.1, C30.1, C31.1, C32.1
- net RA10: now reaches U1.49 (P49)
- net AccA16 renamed RA8
- net AccA17 renamed RA7
- net AccA18 renamed RA6
- net AccA19 renamed RA5
- net AccA20 renamed RA4
- net AccA21 renamed RA3
- net AccA22 renamed RA2
- net AccA23 renamed RA1
- net AccD~LE~: no longer names the net of U1.7 (P7)
- net AccD~OE~: no longer names the net of U1.8 (P8)
- net AccE: no longer names the net of U1.82 (P82)
- net Acc~VMA~: no longer names the net of U1.76 (P76)
- net C20M: no longer names the net of U1.22 (I/O/GCK1)
- net MacA17: no longer names the net of U1.17 (P17)
- net MacA18: no longer names the net of U1.16 (P16)
- net MacA19: no longer names the net of U1.15 (P15)
- net MacA20: no longer names the net of U1.14 (P14)
- net MacA21: no longer names the net of U1.13 (P13)
- net MacA22: no longer names the net of U1.12 (P12)
- net MacA23: no longer names the net of U1.11 (P11)
- net MacA~LE~: no longer names the net of U1.2 (I/O/GTS4)
- net MacA~OE~: no longer names the net of U1.3 (I/O/GTS1)
- net MacD~LE~: no longer names the net of U1.4 (I/O/GTS2)
- net MacD~OE~: no longer names the net of U1.6 (P6)
- net MacR~W~: no longer names the net of U1.18 (P18)
- net MacR~W~: no longer U1.34 (P34)
- net RAM01~CS~: no longer names the net of U1.55 (P55)
- net RAM23~CS~: no longer names the net of U1.56 (P56)
- net RAML~CS~: no longer names the net of U1.60 (P60)
- net RAMU~CS~: no longer names the net of U1.61 (P61)
- net RAM~CS~: no longer names the net of U1.52 (P52)
- net RL~CS~: no longer names the net of U1.85 (P85)
- net RU~CS~: no longer names the net of U1.86 (P86)
- net ~PMCYC~: no longer names the net of U1.95 (P95)
- net ~R~W: no longer names the net of U1.53 (P53)
- new net RA0: U1.34 (P34)
- new net RA11: U1.50 (P50)
- new net RA9: U1.46 (P46)
Other:
- moved on the sheet: U1

Commit message: more
Connections:
- net A1: now also U1.94 (P94)
- net A10: now also U1.8 (P8)
- net A11: now also U1.9 (P9)
- net A12: now also U1.10 (P10)
- net A13: now also U1.11 (P11)
- net A14: now also U1.12 (P12)
- net A15: now also U1.13 (P13)
- net A16: now also U1.14 (P14)
- net A17: now also U1.15 (P15)
- net A18: now also U1.16 (P16)
- net A19: now also U1.17 (P17)
- net A2: now also U1.95 (P95)
- net A20: now also U1.18 (P18)
- net A21: now also U1.19 (P19)
- net A22: now also U1.20 (P20)
- net A23: now also U1.24 (P24)
- net A3: now also U1.96 (P96)
- net A4: now also U1.97 (P97)
- net A5: now also U1.2 (I/O/GTS4)
- net A6: now also U1.3 (I/O/GTS1)
- net A7: now also U1.4 (I/O/GTS2)
- net A8: now also U1.6 (P6)
- net A9: now also U1.7 (P7)
- net ADoutLE0: now also U1.85 (P85)
- net ADoutLE1: now also U1.82 (P82)
- net AccR~W~: now also U1.29 (P29)
- net Acc~AS~: now also U1.33 (P33)
- net Acc~BERR~: now also U1.92 (P92)
- net Acc~DTACK: now also U1.28 (P28)
- net Acc~LDS~: now also U1.30 (P30)
- net Acc~UDS~: now also U1.32 (P32)
- net Acc~VPA~: now also U1.93 (P93)
- net Aout~OE~: now also U1.87 (P87)
- net C16M: now also U1.22 (I/O/GCK1)
- net C8M: now also U1.23 (I/O/GCK2)
- net DinLE: now also U1.86 (P86)
- net Din~OE~: now also U1.90 (P90)
- net Dout~OE~: now also U1.89 (P89)
- net FCLK: now also U1.27 (I/O/GCK3)
- net L~WE~: now also U1.56 (P56)
- net MacE: now also U1.25 (P25)
- net Mac~AS~: now also U1.81 (P81)
- net Mac~BERR~: now also U1.74 (P74)
- net Mac~DTACK~: now also U1.78 (P78)
- net Mac~LDS~: now also U1.79 (P79)
- net Mac~UDS~: now also U1.80 (P80)
- net Mac~VMA~: now also U1.77 (P77)
- net Mac~VPA~: now also U1.76 (P76)
- net RA0: now also U1.37 (P37); no longer U1.34 (P34)
- net RA1: now also U1.39 (P39); no longer U1.35 (P35)
- net RA10: now also U1.53 (P53); no longer U1.49 (P49)
- net RA11: now also U1.54 (P54); no longer U1.50 (P50)
- net RA2: now also U1.40 (P40); no longer U1.36 (P36)
- net RA3: now also U1.41 (P41); no longer U1.37 (P37)
- net RA4: now also U1.42 (P42); no longer U1.39 (P39)
- net RA5: now also U1.43 (P43); no longer U1.40 (P40)
- net RA6: now also U1.46 (P46); no longer U1.41 (P41)
- net RA7: now also U1.49 (P49); no longer U1.42 (P42)
- net RA8: now also U1.50 (P50); no longer U1.43 (P43)
- net RA9: now also U1.52 (P52); no longer U1.46 (P46)
- net ROM~CS~: now also U1.34 (P34)
- net U~WE~: now also U1.55 (P55)
- net ~CAS~: now also U1.35 (P35)
- net ~OE~: now also U1.36 (P36)
- net ~RAS~: now also U1.58 (P58)
- net ~RESET~: now also U1.91 (P91)
- net ~RESET~r: now also U1.1 (I/O/GTS3), U1.99 (I/O/GSR)
