File: SE-030.sch (KiCad schematic (older format))
At the start: 30 parts

Commit message: idk
Connections:
- wire segments 119 -> 120

Commit message: Much progress
Parts:
- removed C10, C11, C12, C13, C14, C15, C17, C18, C20, C21, C22, C23, C24, C25, C26, C27, C28, C7, C8, C9: 2u2, stdpads:C_0603, symbol Device:C_Small
- removed C29: 10u, stdpads:C_0805, symbol Device:C_Small
Connections:
- net labels removed: +3V3, +5V
- wire segments 120 -> 64
- no-connect marks 0 -> 2
Other:
- moved on the sheet: FID1, FID2, FID3, FID4, H1, H2, H3, H4, H5

Commit message: more
Changed lines of the file:
@@
 Wire Wire Line
 	2700 3300 3200 3300
-Wire Wire Line
-	3100 1600 3100 1700
 Connection ~ 3100 1600
 Connection ~ 2800 2700
@@
 Wire Wire Line
 	3100 2900 3200 2900
-Connection ~ 3100 1700
 Wire Wire Line
 	2700 3400 3200 3400
@@
 	3000 1400 3000 2450
 Connection ~ 3000 2450
-Wire Wire Line
-	3100 1700 3100 2900
 Wire Wire Line
 	4500 2700 4500 2500
@@
 	4200 1900 4600 1900
 Wire Wire Line
-	3200 1700 3100 1700
-Wire Wire Line
 	3100 1600 3200 1600
 Wire Wire Line
@@
 F9 "~VPA~" I R 4200 1700 50
 F10 "~RESET~" B L 3200 1600 50
-F11 "~HALT~" B L 3200 1700 50
-F12 "~BERR~" I R 4200 1900 50
-F13 "~IPL~0" I L 3200 1900 50
-F14 "~IPL~1" I L 3200 2000 50
-F15 "~IPL~2" I L 3200 2100 50
-F16 "CLK" I R 4200 2100 50
+F11 "~BERR~" I R 4200 1900 50
+F12 "~IPL~0" I L 3200 1900 50
+F13 "~IPL~1" I L 3200 2000 50
+F14 "~IPL~2" I L 3200 2100 50
+F15 "CLK" I R 4200 2100 50
 $EndSheet
 Wire Bus Line
@@
 Wire Bus Line
 	2800 2350 4400 2350
+Wire Wire Line
+	3100 1600 3100 2900
 $EndSCHEMATC
