File: Buf.sch (KiCad schematic (older format))
At the start: 7 parts

Commit message: idk
Parts:
- removed U?: 74AHCT573, symbol GW_Logic:74573
- U? (x2): value 74AHC573 -> 74AHCT573
Changed lines of the file:
@@
-$EndComp
-$Comp
-L GW_Logic:74573 U?
-U 1 1 609454C2
-P 2400 4050
-F 0 "U?" H 2400 4650 50  0000 C CNN
-F 1 "74AHCT573" V 2400 4050 50  0000 C CNN
-F 2 "" H 2400 3400 50  0001 C TNN
-F 3 "" H 2400 4150 60  0001 C CNN
-	1    2400 4050
-	-1   0    0    -1
 $EndComp
 $Comp
@@
 $EndComp
 $Comp
-L power:GND #PWR?
-U 1 1 60952C35
-P 2800 4500
-F 0 "#PWR?" H 2800 4250 50  0001 C CNN
-F 1 "GND" H 2805 4327 50  0000 C CNN
-F 2 "" H 2800 4500 50  0001 C CNN
-F 3 "" H 2800 4500 50  0001 C CNN
-	1    2800 4500
-	1    0    0    -1
-$EndComp
-$Comp
 L power:+3V3 #PWR?
 U 1 1 609530BF
@@
 	1    0    0    -1
 $EndComp
-$Comp
-L power:+3V3 #PWR?
-U 1 1 60953C96
-P 2000 3600
-F 0 "#PWR?" H 2000 3450 50  0001 C CNN
-F 1 "+3V3" H 2000 3750 50  0000 C CNN
-F 2 "" H 2000 3600 50  0001 C CNN
-F 3 "" H 2000 3600 50  0001 C CNN
-	1    2000 3600
-	1    0    0    -1
-$EndComp
 Text HLabel 2800 1200 2    50   Input ~ 0
 MacA~OE~
 Text HLabel 2800 2400 2    50   Input ~ 0
 MacA~OE~
-Text HLabel 2800 3600 2    50   Input ~ 0
-MacA~OE~
-Text HLabel 2000 4500 0    50   Input ~ 0
-MacA~LE~
 Text HLabel 2000 3300 0    50   Input ~ 0
 MacA~LE~
-Text Label 2800 3800 0    50   ~ 0
-AccA18
-Wire Wire Line
-	2800 4300 3100 4300
-Wire Wire Line
-	2800 4200 3100 4200
-Wire Wire Line
-	2800 4100 3100 4100
-Wire Wire Line
-	2800 4000 3100 4000
-Wire Wire Line
-	2800 3900 3100 3900
-Wire Wire Line
-	2800 3800 3100 3800
-Wire Wire Line
-	2800 3700 3100 3700
-Entry Wire Line
-	3100 4300 3200 4400
-Entry Wire Line
-	3100 4200 3200 4300
-Entry Wire Line
-	3100 4100 3200 4200
-Entry Wire Line
-	3100 4000 3200 4100
-Entry Wire Line
-	3100 3900 3200 4000
-Entry Wire Line
-	3100 3800 3200 3900
-Entry Wire Line
-	3100 3700 3200 3800
-Text Label 2800 3700 0    50   ~ 0
-AccA17
-Text Label 2800 3900 0    50   ~ 0
-AccA19
-Text Label 2800 4000 0    50   ~ 0
-AccA20
-Text Label 2800 4100 0    50   ~ 0
-AccA21
-Text Label 2800 4200 0    50   ~ 0
-AccA22
-Text Label 2800 4300 0    50   ~ 0
-AccA23
 Text Label 2800 3200 0    50   ~ 0
 AccA16
@@
 	2000 2500 1700 2500
 Entry Wire Line
-	1700 4300 1600 4400
-Entry Wire Line
-	1700 4200 1600 4300
-Entry Wire Line
-	1700 4100 1600 4200
-Entry Wire Line
-	1700 4000 1600 4100
-Entry Wire Line
-	1700 3900 1600 4000
-Entry Wire Line
-	1700 3800 1600 3900
-Entry Wire Line
-	1700 3700 1600 3800
-Entry Wire Line
 	1700 2500 1600 2600
 Entry Wire Line
@@
 Text HLabel 2000 2100 0    50   Input ~ 0
 MacA~LE~
-Text Label 2000 3800 2    50   ~ 0
-MacA18
-Wire Wire Line
-	2000 4300 1700 4300
-Wire Wire Line
-	2000 4200 1700 4200
-Wire Wire Line
-	2000 4100 1700 4100
-Wire Wire Line
-	2000 4000 1700 4000
-Wire Wire Line
-	2000 3900 1700 3900
-Wire Wire Line
-	2000 3800 1700 3800
-Wire Wire Line
-	2000 3700 1700 3700
-Text Label 2000 3700 2    50   ~ 0
-MacA17
-Text Label 2000 3900 2    50   ~ 0
-MacA19
-Text Label 2000 4000 2    50   ~ 0
-MacA20
-Text Label 2000 4100 2    50   ~ 0
-MacA21
-Text Label 2000 4200 2    50   ~ 0
-MacA22
-Text Label 2000 4300 2    50   ~ 0
-MacA23
 Text HLabel 1600 1400 0    50   BiDi ~ 0
 MacA[23..1]
@@
 P 5150 3450
 F 0 "U?" H 5150 4050 50  0000 C CNN
-F 1 "74AHC573" V 5150 3450 50  0000 C CNN
+F 1 "74AHCT573" V 5150 3450 50  0000 C CNN
 F 2 "" H 5150 2800 50  0001 C TNN
 F 3 "" H 5150 3550 60  0001 C CNN
@@
 P 5150 6050
 F 0 "U?" H 5150 6650 50  0000 C CNN
-F 1 "74AHC573" V 5150 6050 50  0000 C CNN
+F 1 "74AHCT573" V 5150 6050 50  0000 C CNN
 F 2 "" H 5150 5400 50  0001 C TNN
 F 3 "" H 5150 6150 60  0001 C CNN
@@
 	4300 1900 4350 1900
 Wire Bus Line
-	3200 1400 3200 4400
+	3200 1400 3200 3300
 Wire Bus Line
-	1600 1400 1600 4400
+	1600 1400 1600 3300
 Wire Bus Line
 	4350 1900 4350 6500
 Wire Bus Line
 	5950 1900 5950 6500
-Text HLabel 2800 4400 2    50   Input ~ 0
-AccR~W~
-Text HLabel 2000 4400 0    50   Input ~ 0
-MacR~W~
 $EndSCHEMATC

Commit message: Much progress
Parts:
- added C33, C34, C35, C36, C37, C38, C39, C40, C41, C42, C43, C44: 2u2, stdpads:C_0603, symbol Device:C_Small
- added U16, U17, U18, U2, U23, U24: 74AHCT573, stdpads:TSSOP-20_4.4x6.5mm_P0.65mm, symbol GW_Logic:74573
- U13, U15, U19, U20, U21, U22: renamed from U?; footprint (none) -> stdpads:TSSOP-20_4.4x6.5mm_P0.65mm
Connections:
- net MacA~LE~ is gone; now on net ADoutLE0: U13.11 (~LE~), U15.11 (~LE~)
- net +3V3: now also C33.1, C34.1, C35.1, C36.1, C37.1, C38.1, C39.1, C40.1, C41.1, C42.1, C43.1, C44.1; no longer U13.20 (Vcc), U15.20 (Vcc), U19.20 (Vcc), U20.20 (Vcc), U21.20 (Vcc), U22.20 (Vcc)
- net AccA1: now also U17.9 (D7); no longer U13.2 (D0)
- net AccA10: now also U18.8 (D6); no longer U15.3 (D1)
- net AccA11: now also U18.7 (D5); no longer U15.4 (D2)
- net AccA12: now also U18.6 (D4); no longer U15.5 (D3)
- net AccA13: now also U18.5 (D3); no longer U15.6 (D4)
- net AccA14: now also U18.4 (D2); no longer U15.7 (D5)
- net AccA15: now also U18.3 (D1); no longer U15.8 (D6)
- net AccA16: now also U18.2 (D0); no longer U15.9 (D7)
- net AccA2: now also U17.8 (D6); no longer U13.3 (D1)
- net AccA3: now also U17.7 (D5); no longer U13.4 (D2)
- net AccA4: now also U17.6 (D4); no longer U13.5 (D3)
- net AccA5: now also U17.5 (D3); no longer U13.6 (D4)
- net AccA6: now also U17.4 (D2); no longer U13.7 (D5)
- net AccA7: now also U17.3 (D1); no longer U13.8 (D6)
- net AccA8: now also U17.2 (D0); no longer U13.9 (D7)
- net AccA9: now also U18.9 (D7); no longer U15.2 (D0)
- net AccD0: now also U20.12 (Q7), U23.9 (D7); no longer U19.2 (D0), U20.19 (Q0)
- net AccD1: now also U20.13 (Q6), U23.8 (D6); no longer U19.3 (D1), U20.18 (Q1)
- net AccD10: now also U22.14 (Q5), U24.7 (D5); no longer U21.4 (D2), U22.17 (Q2)
- net AccD11: now also U22.15 (Q4), U24.6 (D4); no longer U21.5 (D3), U22.16 (Q3)
- net AccD12: now also U22.16 (Q3), U24.5 (D3); no longer U21.6 (D4), U22.15 (Q4)
- net AccD13: now also U22.17 (Q2), U24.4 (D2); no longer U21.7 (D5), U22.14 (Q5)
- net AccD14: now also U22.18 (Q1), U24.3 (D1); no longer U21.8 (D6), U22.13 (Q6)
- net AccD15: now also U22.19 (Q0), U24.2 (D0); no longer U21.9 (D7), U22.12 (Q7)
- net AccD2: now also U20.14 (Q5), U23.7 (D5); no longer U19.4 (D2), U20.17 (Q2)
- net AccD3: now also U20.15 (Q4), U23.6 (D4); no longer U19.5 (D3), U20.16 (Q3)
- net AccD4: now also U20.16 (Q3), U23.5 (D3); no longer U19.6 (D4), U20.15 (Q4)
- net AccD5: now also U20.17 (Q2), U23.4 (D2); no longer U19.7 (D5), U20.14 (Q5)
- net AccD6: now also U20.18 (Q1), U23.3 (D1); no longer U19.8 (D6), U20.13 (Q6)
- net AccD7: now also U20.19 (Q0), U23.2 (D0); no longer U19.9 (D7), U20.12 (Q7)
- net AccD8: now also U22.12 (Q7), U24.9 (D7); no longer U21.2 (D0), U22.19 (Q0)
- net AccD9: now also U22.13 (Q6), U24.8 (D6); no longer U21.3 (D1), U22.18 (Q1)
- net GND: now also C33.2, C34.2, C35.2, C36.2, C37.2, C38.2, C39.2, C40.2, C41.2, C42.2, C43.2, C44.2, U16.10 (GND), U17.1 (~OE~), U17.10 (GND), U18.1 (~OE~), U18.10 (GND), U2.1 (~OE~), U2.10 (GND), U23.1 (~OE~), U23.10 (GND), U24.1 (~OE~), U24.10 (GND)
- net MacA1: now also U13.12 (Q7); no longer U13.19 (Q0)
- net MacA10: now also U15.13 (Q6); no longer U15.18 (Q1)
- net MacA11: now also U15.14 (Q5); no longer U15.17 (Q2)
- net MacA12: now also U15.15 (Q4); no longer U15.16 (Q3)
- net MacA13: now also U15.16 (Q3); no longer U15.15 (Q4)
- net MacA14: now also U15.17 (Q2); no longer U15.14 (Q5)
- net MacA15: now also U15.18 (Q1); no longer U15.13 (Q6)
- net MacA16: now also U15.19 (Q0); no longer U15.12 (Q7)
- net MacA2: now also U13.13 (Q6); no longer U13.18 (Q1)
- net MacA3: now also U13.14 (Q5); no longer U13.17 (Q2)
- net MacA4: now also U13.15 (Q4); no longer U13.16 (Q3)
- net MacA5: now also U13.16 (Q3); no longer U13.15 (Q4)
- net MacA6: now also U13.17 (Q2); no longer U13.14 (Q5)
- net MacA7: now also U13.18 (Q1); no longer U13.13 (Q6)
- net MacA8: now also U13.19 (Q0); no longer U13.12 (Q7)
- net MacA9: now also U15.12 (Q7); no longer U15.19 (Q0)
- net MacD0: now also U19.12 (Q7), U20.9 (D7); no longer U19.19 (Q0), U20.2 (D0)
- net MacD1: now also U19.13 (Q6), U20.8 (D6); no longer U19.18 (Q1), U20.3 (D1)
- net MacD10: now also U21.14 (Q5), U22.7 (D5); no longer U21.17 (Q2), U22.4 (D2)
- net MacD11: now also U21.15 (Q4), U22.6 (D4); no longer U21.16 (Q3), U22.5 (D3)
- net MacD12: now also U21.16 (Q3), U22.5 (D3); no longer U21.15 (Q4), U22.6 (D4)
- net MacD13: now also U21.17 (Q2), U22.4 (D2); no longer U21.14 (Q5), U22.7 (D5)
- net MacD14: now also U21.18 (Q1), U22.3 (D1); no longer U21.13 (Q6), U22.8 (D6)
- net MacD15: now also U21.19 (Q0), U22.2 (D0); no longer U21.12 (Q7), U22.9 (D7)
- net MacD2: now also U19.14 (Q5), U20.7 (D5); no longer U19.17 (Q2), U20.4 (D2)
- net MacD3: now also U19.15 (Q4), U20.6 (D4); no longer U19.16 (Q3), U20.5 (D3)
- net MacD4: now also U19.16 (Q3), U20.5 (D3); no longer U19.15 (Q4), U20.6 (D4)
- net MacD5: now also U19.17 (Q2), U20.4 (D2); no longer U19.14 (Q5), U20.7 (D5)
- net MacD6: now also U19.18 (Q1), U20.3 (D1); no longer U19.13 (Q6), U20.8 (D6)
- net MacD7: now also U19.19 (Q0), U20.2 (D0); no longer U19.12 (Q7), U20.9 (D7)
- net MacD8: now also U21.12 (Q7), U22.9 (D7); no longer U21.19 (Q0), U22.2 (D0)
- net MacD9: now also U21.13 (Q6), U22.8 (D6); no longer U21.18 (Q1), U22.3 (D1)
- net AccD~LE~ renamed ADoutLE0
- net ADoutLE0: now also U16.11 (~LE~)
- net AccD~OE~ renamed Din~OE~
- net MacA~OE~ renamed Aout~OE~
- net Aout~OE~: now also U16.1 (~OE~)
- net MacD~LE~ renamed DinLE
- net MacD~OE~ renamed Dout~OE~
- new net: U13.2 (D0), U17.19 (Q0)
- new net: U13.3 (D1), U17.18 (Q1)
- new net: U13.4 (D2), U17.17 (Q2)
- new net: U13.5 (D3), U17.16 (Q3)
- new net: U13.6 (D4), U17.15 (Q4)
- new net: U13.7 (D5), U17.14 (Q5)
- new net: U13.8 (D6), U17.13 (Q6)
- new net: U13.9 (D7), U17.12 (Q7)
- new net: U15.2 (D0), U18.19 (Q0)
- new net: U15.3 (D1), U18.18 (Q1)
- new net: U15.4 (D2), U18.17 (Q2)
- new net: U15.5 (D3), U18.16 (Q3)
- new net: U15.6 (D4), U18.15 (Q4)
- new net: U15.7 (D5), U18.14 (Q5)
- new net: U15.8 (D6), U18.13 (Q6)
- new net: U15.9 (D7), U18.12 (Q7)
- new net: U19.2 (D0), U23.19 (Q0)
- new net: U19.3 (D1), U23.18 (Q1)
- new net: U19.4 (D2), U23.17 (Q2)
- new net: U19.5 (D3), U23.16 (Q3)
- new net: U19.6 (D4), U23.15 (Q4)
- new net: U19.7 (D5), U23.14 (Q5)
- new net: U19.8 (D6), U23.13 (Q6)
- new net: U19.9 (D7), U23.12 (Q7)
- new net: U21.2 (D0), U24.19 (Q0)
- new net: U21.3 (D1), U24.18 (Q1)
- new net: U21.4 (D2), U24.17 (Q2)
- new net: U21.5 (D3), U24.16 (Q3)
- new net: U21.6 (D4), U24.15 (Q4)
- new net: U21.7 (D5), U24.14 (Q5)
- new net: U21.8 (D6), U24.13 (Q6)
- new net: U21.9 (D7), U24.12 (Q7)
- new net: U16.2 (D0), U2.19 (Q0)
- new net: U16.3 (D1), U2.18 (Q1)
- new net: U16.4 (D2), U2.17 (Q2)
- new net: U16.5 (D3), U2.16 (Q3)
- new net: U16.6 (D4), U2.15 (Q4)
- new net: U16.7 (D5), U2.14 (Q5)
- new net: U16.8 (D6), U2.13 (Q6)
- new net: U16.9 (D7), U2.12 (Q7)
- new net +5V: U13.20 (Vcc), U15.20 (Vcc), U16.20 (Vcc), U17.20 (Vcc), U18.20 (Vcc), U19.20 (Vcc), U2.20 (Vcc), U20.20 (Vcc), U21.20 (Vcc), U22.20 (Vcc), U23.20 (Vcc), U24.20 (Vcc)
- new net ADoutLE1: U17.11 (~LE~), U18.11 (~LE~), U2.11 (~LE~), U23.11 (~LE~), U24.11 (~LE~)
- new net AccA17: U2.8 (D6)
- new net AccA18: U2.7 (D5)
- new net AccA19: U2.6 (D4)
- new net AccA20: U2.5 (D3)
- new net AccA21: U2.4 (D2)
- new net AccA22: U2.3 (D1)
- new net AccA23: U2.2 (D0)
- new net Acc~R~W: U2.9 (D7)
- new net MacA17: U16.13 (Q6)
- new net MacA18: U16.14 (Q5)
- new net MacA19: U16.15 (Q4)
- new net MacA20: U16.16 (Q3)
- new net MacA21: U16.17 (Q2)
- new net MacA22: U16.18 (Q1)
- new net MacA23: U16.19 (Q0)
- new net Mac~R~W: U16.12 (Q7)
Other:
- moved on the sheet: U13, U15, U19, U20, U21, U22

Commit message: Add LC... sloppy
Connections:
- net +3V3 is gone; now on net +5V: C33.1, C34.1, C35.1, C36.1, C37.1, C38.1, C39.1, C40.1, C41.1, C42.1, C43.1, C44.1
Other:
- moved on the sheet: C33, C34, C35, C36, C37, C38, C39, C40, C41, C42, C43, C44
