File: Clk.sch (KiCad schematic (older format))
At the start: 11 parts, among them SW1 OSCSEL, U4 20M, U5 25M

Commit message: Add LC... sloppy
Parts:
- removed C7: 2u2, stdpads:C_0603, symbol Device:C_Small
- removed R10, R11: 10k, stdpads:R_0603, symbol Device:R_Small
- removed R12: 22, stdpads:R_0603, symbol Device:R_Small
- removed SW1: OSCSEL, stdpads:SW_DIP_SPSTx02_Slide_DSHP02TS_P1.27mm, symbol Switch:SW_DIP_x02
Connections:
- net CK20EN: now reaches U4.1 (EN)
- net CK25EN: now reaches U5.1 (EN)
