File: MC68k.sch (KiCad schematic (older format))
At the start: 1 part, among them U14 MC68000FN

Commit message: idk
Parts:
- U14: footprint Package_LCC:PLCC-68 -> stdpads:PLCC-68_SMDSocket
Connections:
- net A1: now also U14.32 (A1)
- net A10: now also U14.41 (A10)
- net A11: now also U14.42 (A11)
- net A12: now also U14.43 (A12)
- net A13: now also U14.44 (A13)
- net A14: now also U14.45 (A14)
- net A15: now also U14.46 (A15)
- net A16: now also U14.47 (A16)
- net A17: now also U14.48 (A17)
- net A18: now also U14.49 (A18)
- net A19: now also U14.50 (A19)
- net A2: now also U14.33 (A2)
- net A20: now also U14.51 (A20)
- net A21: now also U14.53 (A21)
- net A22: now also U14.54 (A22)
- net A23: now also U14.55 (A23)
- net A3: now also U14.34 (A3)
- net A4: now also U14.35 (A4)
- net A5: now also U14.36 (A5)
- net A6: now also U14.37 (A6)
- net A7: now also U14.38 (A7)
- net A8: now also U14.39 (A8)
- net A9: now also U14.40 (A9)
- net CLK: now also U14.15 (CLK)
- net D0: now also U14.5 (D0)
- net D1: now also U14.4 (D1)
- net D10: now also U14.63 (D10)
- net D11: now also U14.62 (D11)
- net D12: now also U14.61 (D12)
- net D13: now also U14.60 (D13)
- net D14: now also U14.59 (D14)
- net D15: now also U14.58 (D15)
- net D2: now also U14.3 (D2)
- net D3: now also U14.2 (D3)
- net D4: now also U14.1 (D4)
- net D5: now also U14.68 (D5)
- net D6: now also U14.67 (D6)
- net D7: now also U14.66 (D7)
- net D8: now also U14.65 (D8)
- net D9: now also U14.64 (D9)
- net E: now also U14.22 (E)
- net R~W~: now also U14.9 (R/W)
- net ~AS~: now also U14.6 (AS)
- net ~BERR~: now also U14.24 (BERR)
- net ~DTACK~: now also U14.10 (DTACK)
- net ~HALT~: now also U14.19 (HALT)
- net ~IPL~0: now also U14.27 (IPL0)
- net ~IPL~1: now also U14.26 (IPL1)
- net ~IPL~2: now also U14.25 (IPL2)
- net ~LDS~: now also U14.8 (LDS)
- net ~RESET~: now also U14.20 (RESET)
- net ~UDS~: now also U14.7 (UDS)
- net ~VMA~: now also U14.21 (VMA)
- net ~VPA~: now also U14.23 (VPA)
- net +5V: now reaches U14.12 (BGACK)
- net +5V: now also U14.13 (BR), U14.14 (VCC), U14.52 (VCC)
- net GND: now reaches U14.16 (GND)
- net GND: now also U14.17 (GND), U14.56 (GND), U14.57 (GND)
- no-connect marks 0 -> 4

Commit message: Much progress
Parts:
- added C1, C2, C3, C4: 10u, stdpads:C_0805, symbol Device:C_Small
- U14: value MC68000FN -> MC68HC000FN20; footprint stdpads:PLCC-68_SMDSocket -> Package_LCC:PLCC-68_SMD-Socket
Connections:
- net +5V: now also C1.1, C2.1, C3.1, C4.1
- net GND: now also C1.2, C2.2, C3.2, C4.2
- net E: no longer names the net of U14.22 (E)
- net ~VMA~: no longer names the net of U14.21 (VMA)
Other:
- moved on the sheet: U14

Commit message: more
Connections:
- net ~HALT~ is gone; now on net ~RESET~: U14.19 (HALT)
Changed lines of the file:
@@
 Text HLabel 3650 1500 2    50   Output ~ 0
 A[23..1]
-Text HLabel 1300 4800 0    50   BiDi ~ 0
-~HALT~
 NoConn ~ 1300 2600
 NoConn ~ 1300 2700
@@
 Connection ~ 2100 7200
 Connection ~ 1700 7200
+Wire Wire Line
+	1300 4800 1300 5000
 Wire Bus Line
 	3600 3900 3600 5400

Commit message: Add LC... sloppy
Parts:
- removed C3, C4: 10u, stdpads:C_0805, symbol Device:C_Small
- U14: footprint Package_LCC:PLCC-68_SMD-Socket -> stdpads:PLCC-68
Connections:
- no-connect marks 4 -> 6
Changed lines of the file:
@@
 $Descr A4 11693 8268
 encoding utf-8
-Sheet 7 7
+Sheet 5 10
 Title ""
 Date ""
@@
 F 0 "U14" H 2300 5650 50  0000 C CNN
 F 1 "MC68HC000FN20" H 2300 5550 50  0000 C CNN
-F 2 "Package_LCC:PLCC-68_SMD-Socket" H 1550 5850 50  0001 C CNN
+F 2 "stdpads:PLCC-68" H 1550 5850 50  0001 C CNN
 F 3 "http://www.nxp.com/files/32bit/doc/ref_manual/MC68000UM.pdf" H 2300 3600 50  0001 C CNN
 	1    2300 3600
@@
 Wire Wire Line
 	1300 7400 1700 7400
-Connection ~ 2500 7400
-Wire Wire Line
-	2100 7200 2500 7200
-$Comp
-L Device:C_Small C?
-U 1 1 613F0B66
-P 2500 7300
-AR Path="/613F0B66" Ref="C?"  Part="1"
-AR Path="/60D70CB4/613F0B66" Ref="C?"  Part="1"
-AR Path="/5F72F108/613F0B66" Ref="C4"  Part="1"
-F 0 "C4" H 2550 7350 50  0000 L CNN
-F 1 "10u" H 2550 7250 50  0000 L CNN
-F 2 "stdpads:C_0805" H 2500 7300 50  0001 C CNN
-F 3 "~" H 2500 7300 50  0001 C CNN
-	1    2500 7300
-	1    0    0    -1
-$EndComp
-$Comp
-L Device:C_Small C?
-U 1 1 613F0B6D
-P 2100 7300
-AR Path="/613F0B6D" Ref="C?"  Part="1"
-AR Path="/60D70CB4/613F0B6D" Ref="C?"  Part="1"
-AR Path="/5F72F108/613F0B6D" Ref="C3"  Part="1"
-F 0 "C3" H 2150 7350 50  0000 L CNN
-F 1 "10u" H 2150 7250 50  0000 L CNN
-F 2 "stdpads:C_0805" H 2100 7300 50  0001 C CNN
-F 3 "~" H 2100 7300 50  0001 C CNN
-	1    2100 7300
-	1    0    0    -1
-$EndComp
-$Comp
-L power:GND #PWR?
-U 1 1 613F0B73
-P 2500 7400
-AR Path="/5F723900/613F0B73" Ref="#PWR?"  Part="1"
-AR Path="/60D70CB4/613F0B73" Ref="#PWR?"  Part="1"
-AR Path="/613F0B73" Ref="#PWR?"  Part="1"
-AR Path="/5F72F108/613F0B73" Ref="#PWR0105"  Part="1"
-F 0 "#PWR0105" H 2500 7150 50  0001 C CNN
-F 1 "GND" H 2500 7250 50  0000 C CNN
-F 2 "" H 2500 7400 50  0001 C CNN
-F 3 "" H 2500 7400 50  0001 C CNN
-	1    2500 7400
-	1    0    0    -1
-$EndComp
-Wire Wire Line
-	2100 7400 2500 7400
-Wire Wire Line
-	1700 7400 2100 7400
+Wire Wire Line
+	1300 4800 1300 5000
+NoConn ~ 1300 3100
+NoConn ~ 1300 3200
+$Comp
+L power:GND #PWR0126
+U 1 1 61B1134E
+P 1700 7400
+F 0 "#PWR0126" H 1700 7150 50  0001 C CNN
+F 1 "GND" H 1700 7250 50  0000 C CNN
+F 2 "" H 1700 7400 50  0001 C CNN
+F 3 "" H 1700 7400 50  0001 C CNN
+	1    1700 7400
+	1    0    0    -1
+$EndComp
 Connection ~ 1700 7400
-Connection ~ 2100 7400
-Wire Wire Line
-	2100 7200 1700 7200
-Connection ~ 2100 7200
-Connection ~ 1700 7200
-Wire Wire Line
-	1300 4800 1300 5000
 Wire Bus Line
 	3600 3900 3600 5400
