File: PDS.sch (KiCad schematic (older format))
At the start: 1 part, among them J1 MacSEPDS

Commit message: idk
Parts:
- J1: symbol SE-030-rescue:MacSEPDS-GW_Connector -> GW_Connector:MacSEPDS
Connections:
- net +5V: no longer J1.B14 (+5V), J1.B15 (+5V), J1.B16 (+5V)
- net GND: no longer J1.B2 (GND), J1.B3 (GND), J1.B4 (GND), J1.B5 (GND), J1.B6 (GND), J1.B7 (GND), J1.B8 (GND)
- net ~EXT.DTK~: no longer names the net of J1.B28 (~EXT.DTK~)
- no-connect marks 19 -> 20
Changed lines of the file:
@@
 $EndDescr
 $Comp
-L SE-030-rescue:MacSEPDS-GW_Connector J?
+L GW_Connector:MacSEPDS J?
 U 1 1 5F6DD05A
 P 1350 3950
@@
 $EndComp
 $Comp
-L SE-030-rescue:MacSEPDS-GW_Connector J?
+L GW_Connector:MacSEPDS J?
 U 3 1 5F6E0CCF
 P 3900 3950
@@
 Text HLabel 2750 4350 2    50   Output ~ 0
 ~BERR~
-Text HLabel 2750 5050 2    50   Input ~ 0
-~EXT.DTK~
 Text HLabel 1500 4900 2    50   Output ~ 0
 E
@@
 Text Label 1500 4800 0    50   ~ 0
 A23
-Connection ~ 2750 3550
-Connection ~ 2750 3150
-Connection ~ 2750 3050
-Wire Wire Line
-	2750 3050 2750 3150
-Wire Wire Line
-	2750 2950 2750 3050
-Connection ~ 2750 2950
-Connection ~ 2750 2850
-Wire Wire Line
-	2750 2850 2750 2950
-Wire Wire Line
-	2750 2750 2750 2850
-Connection ~ 2750 2750
-Connection ~ 2750 2650
-Wire Wire Line
-	2750 2650 2750 2750
-Wire Wire Line
-	2750 2550 2750 2650
-Connection ~ 2750 2550
-Connection ~ 2750 2450
-Wire Wire Line
-	2750 2450 2750 2550
-Wire Wire Line
-	2750 2350 2750 2450
-Connection ~ 2750 3850
-Wire Wire Line
-	2750 3850 2750 3950
-Wire Wire Line
-	2750 3750 2750 3850
-Connection ~ 2750 3750
-Connection ~ 2750 3650
-Wire Wire Line
-	2750 3650 2750 3750
-Wire Wire Line
-	2750 3650 2750 3550
-$Comp
-L SE-030-rescue:MacSEPDS-GW_Connector J?
+$Comp
+L GW_Connector:MacSEPDS J?
 U 2 1 5F6DF4C8
 P 2600 4000
@@
 	1    0    0    -1
 $EndComp
+Wire Wire Line
+	2750 3550 2750 3950
+Wire Wire Line
+	2750 2350 2750 3150
+NoConn ~ 2750 5050
 Wire Bus Line
 	4350 3700 4350 5200

Commit message: Much progress
Parts:
- added C18, C19, C20, C21, C22, C23, C24, C25: 10u, stdpads:C_0805, symbol Device:C_Small
- J1: footprint (none) -> stdpads:DIN41612_R_3x32_Male_Vertical_THT
Connections:
- net ~BGACK~ is gone; now on net +5V: J1.C4 (~BGACK~)
- net ~BR~ is gone; now on net GND: J1.C3 (~BR~)
- net +5V: now also J1.B14 (+5V), J1.B15 (+5V), J1.B16 (+5V), C18.1, C19.1
- net GND: now also J1.B2 (GND), J1.B3 (GND), J1.B4 (GND), J1.B5 (GND), J1.B6 (GND), J1.B7 (GND), J1.B8 (GND), C18.2, C19.2, C20.2, C21.2, C22.2, C23.2, C24.2, C25.2
- net ~BG~: no longer names the net of J1.C5 (~BG~)
- net ~PMCYC~: no longer names the net of J1.C11 (~PMCYC~)
- new net +12V: C22.1, C23.1
- new net -12V: C24.1, C25.1
- new net -5V: C20.1, C21.1
- no-connect marks 20 -> 22

Commit message: Add LC... sloppy
Parts:
- removed C21, C23, C25: 10u, stdpads:C_0805, symbol Device:C_Small
Connections:
- net +12V: now also J1.A31 (+12V), J1.A32 (+12V), J1.B30 (+12V), J1.B31 (+12V)
- net -12V: now also J1.C32 (-12V)
- net -5V: now also J1.B32 (-5V)
- no-connect marks 22 -> 16
Changed lines of the file:
@@
 $Descr A4 11693 8268
 encoding utf-8
-Sheet 6 7
+Sheet 4 10
 Title ""
 Date ""
@@
 NoConn ~ 1500 2400
 NoConn ~ 1500 2500
-NoConn ~ 1500 5300
-NoConn ~ 1500 5400
-NoConn ~ 2750 5250
-NoConn ~ 2750 5350
-NoConn ~ 2750 5450
 NoConn ~ 2750 4950
 NoConn ~ 2750 4850
@@
 L power:GND #PWR0146
 U 1 1 5F6E485F
-P 4150 5200
-F 0 "#PWR0146" H 4150 4950 50  0001 C CNN
-F 1 "GND" H 4150 5050 50  0000 C CNN
-F 2 "" H 4150 5200 50  0001 C CNN
-F 3 "" H 4150 5200 50  0001 C CNN
-	1    4150 5200
-	1    0    0    -1
-$EndComp
-Wire Wire Line
-	4150 5200 4050 5200
+P 4500 5200
+F 0 "#PWR0146" H 4500 4950 50  0001 C CNN
+F 1 "GND" H 4500 5050 50  0000 C CNN
+F 2 "" H 4500 5200 50  0001 C CNN
+F 3 "" H 4500 5200 50  0001 C CNN
+	1    4500 5200
+	1    0    0    -1
+$EndComp
 NoConn ~ 4050 5300
-NoConn ~ 4050 5400
 $Comp
 L power:GND #PWR0147
 U 1 1 5F6E565A
-P 1600 5200
-F 0 "#PWR0147" H 1600 4950 50  0001 C CNN
-F 1 "GND" H 1600 5050 50  0000 C CNN
-F 2 "" H 1600 5200 50  0001 C CNN
-F 3 "" H 1600 5200 50  0001 C CNN
-	1    1600 5200
-	1    0    0    -1
-$EndComp
-Wire Wire Line
-	1600 5200 1500 5200
+P 1900 5200
+F 0 "#PWR0147" H 1900 4950 50  0001 C CNN
+F 1 "GND" H 1900 5050 50  0000 C CNN
+F 2 "" H 1900 5200 50  0001 C CNN
+F 3 "" H 1900 5200 50  0001 C CNN
+	1    1900 5200
+	1    0    0    -1
+$EndComp
+Wire Wire Line
+	1900 5200 1500 5200
 $Comp
 L power:+5V #PWR0148
@@
 L power:GND #PWR0149
 U 1 1 5F6E6FCB
-P 2850 5150
-F 0 "#PWR0149" H 2850 4900 50  0001 C CNN
-F 1 "GND" H 2850 5000 50  0000 C CNN
-F 2 "" H 2850 5150 50  0001 C CNN
-F 3 "" H 2850 5150 50  0001 C CNN
-	1    2850 5150
-	1    0    0    -1
-$EndComp
-Wire Wire Line
-	2850 5150 2750 5150
+P 3150 5150
+F 0 "#PWR0149" H 3150 4900 50  0001 C CNN
+F 1 "GND" H 3150 5000 50  0000 C CNN
+F 2 "" H 3150 5150 50  0001 C CNN
+F 3 "" H 3150 5150 50  0001 C CNN
+	1    3150 5150
+	1    0    0    -1
+$EndComp
+Wire Wire Line
+	3150 5150 2750 5150
 NoConn ~ 2750 3450
 Text HLabel 4050 2300 2    50   Output ~ 0
@@
 	4050 3600 4250 3600
 Wire Wire Line
-	4050 3500 4450 3500
-Entry Wire Line
-	4250 5100 4350 5200
-Entry Wire Line
-	4250 5000 4350 5100
-Entry Wire Line
-	4250 4900 4350 5000
-Entry Wire Line
-	4250 4800 4350 4900
-Entry Wire Line
-	4250 4700 4350 4800
-Entry Wire Line
-	4250 4600 4350 4700
-Entry Wire Line
-	4250 4500 4350 4600
-Entry Wire Line
-	4250 4400 4350 4500
-Entry Wire Line
-	4250 4300 4350 4400
-Entry Wire Line
-	4250 4200 4350 4300
-Entry Wire Line
-	4250 4100 4350 4200
-Entry Wire Line
-	4250 4000 4350 4100
-Entry Wire Line
-	4250 3900 4350 4000
-Entry Wire Line
-	4250 3800 4350 3900
-Entry Wire Line
-	4250 3700 4350 3800
-Entry Wire Line
-	4250 3600 4350 3700
-Text HLabel 4350 3700 2    50   BiDi ~ 0
-D[15..0]
-Wire Wire Line
 	1500 4100 1700 4100
 Wire Wire Line
@@
 	1    0    0    -1
 $EndComp
-Connection ~ 3300 6400
-$Comp
-L Device:C_Small C?
-U 1 1 616DE7C5
-P 3300 6300
-AR Path="/616DE7C5" Ref="C?"  Part="1"
-AR Path="/5F6DA71D/616DE7C5" Ref="C23"  Part="1"
-F 0 "C23" H 3350 6350 50  0000 L CNN
-F 1 "10u" H 3350 6250 50  0000 L CNN
-F 2 "stdpads:C_0805" H 3300 6300 50  0001 C CNN
-F 3 "~" H 3300 6300 50  0001 C CNN
-	1    3300 6300
-	1    0    0    -1
-$EndComp
 Wire Wire Line
 	1700 6400 2100 6400
@@
 	1    0    0    -1
 $EndComp
-Wire Wire Line
-	2900 6400 3300 6400
 Connection ~ 2900 6400
 $Comp
@@
 F 3 "~" H 1300 6300 50  0001 C CNN
 	1    1300 6300
-	1    0    0    -1
-$EndComp
-Wire Wire Line
-	2500 6400 2900 6400
-Wire Wire Line
-	2100 6400 2500 6400
-Connection ~ 2500 6400
-Wire Wire Line
-	2100 6200 2500 6200
-$Comp
-L Device:C_Small C?
-U 1 1 616DE7F4
-P 2500 6300
-AR Path="/616DE7F4" Ref="C?"  Part="1"
-AR Path="/5F6DA71D/616DE7F4" Ref="C21"  Part="1"
-F 0 "C21" H 2550 6350 50  0000 L CNN
-F 1 "10u" H 2550 6250 50  0000 L CNN
-F 2 "stdpads:C_0805" H 2500 6300 50  0001 C CNN
-F 3 "~" H 2500 6300 50  0001 C CNN
-	1    2500 6300
 	1    0    0    -1
 $EndComp
@@
 	-1   0    0    -1
 $EndComp
-Connection ~ 4100 6400
-$Comp
-L Device:C_Small C?
-U 1 1 616F27A7
-P 4100 6300
-AR Path="/616F27A7" Ref="C?"  Part="1"
-AR Path="/5F6DA71D/616F27A7" Ref="C25"  Part="1"
-F 0 "C25" H 4150 6350 50  0000 L CNN
-F 1 "10u" H 4150 6250 50  0000 L CNN
-F 2 "stdpads:C_0805" H 4100 6300 50  0001 C CNN
-F 3 "~" H 4100 6300 50  0001 C CNN
-	1    4100 6300
-	1    0    0    -1
-$EndComp
 Wire Wire Line
 	3700 6400 4100 6400
 Connection ~ 3700 6400
-Wire Wire Line
-	3700 6200 4100 6200
-Connection ~ 3700 6200
 $Comp
 L Device:C_Small C?
@@
 	1    0    0    -1
 $EndComp
-Wire Wire Line
-	3300 6400 3700 6400
 $Comp
 L power:-5V #PWR0154
@@
 	1    0    0    -1
 $EndComp
-Connection ~ 2100 6200
-Wire Wire Line
-	2900 6200 3300 6200
 $Comp
 L power:+12V #PWR0155
@@
 	1    0    0    -1
 $EndComp
-Connection ~ 2900 6200
 $Comp
 L power:GND #PWR0156
@@
 Connection ~ 2750 3950
 Connection ~ 2750 2350
+Wire Wire Line
+	4050 3500 4450 3500
+Text HLabel 4350 3700 2    50   BiDi ~ 0
+D[15..0]
+Entry Wire Line
+	4250 3600 4350 3700
+Entry Wire Line
+	4250 3700 4350 3800
+Entry Wire Line
+	4250 3800 4350 3900
+Entry Wire Line
+	4250 3900 4350 4000
+Entry Wire Line
+	4250 4000 4350 4100
+Entry Wire Line
+	4250 4100 4350 4200
+Entry Wire Line
+	4250 4200 4350 4300
+Entry Wire Line
+	4250 4300 4350 4400
+Entry Wire Line
+	4250 4400 4350 4500
+Entry Wire Line
+	4250 4500 4350 4600
+Entry Wire Line
+	4250 4600 4350 4700
+Entry Wire Line
+	4250 4700 4350 4800
+Entry Wire Line
+	4250 4800 4350 4900
+Entry Wire Line
+	4250 4900 4350 5000
+Entry Wire Line
+	4250 5000 4350 5100
+Entry Wire Line
+	4250 5100 4350 5200
+Wire Wire Line
+	4050 5200 4300 5200
+Wire Wire Line
+	4300 5200 4300 5250
+Wire Wire Line
+	4300 5250 4400 5250
+Wire Wire Line
+	4400 5250 4400 5200
+Wire Wire Line
+	4400 5200 4500 5200
+$Comp
+L power:-5V #PWR0109
+U 1 1 6176540D
+P 2750 5450
+F 0 "#PWR0109" H 2750 5550 50  0001 C CNN
+F 1 "-5V" H 2750 5600 50  0000 C CNN
+F 2 "" H 2750 5450 50  0001 C CNN
+F 3 "" H 2750 5450 50  0001 C CNN
+	1    2750 5450
+	-1   0    0    1
+$EndComp
+$Comp
+L power:+12V #PWR0110
+U 1 1 6176B64B
+P 1600 5400
+F 0 "#PWR0110" H 1600 5250 50  0001 C CNN
+F 1 "+12V" H 1600 5550 50  0000 C CNN
+F 2 "" H 1600 5400 50  0001 C CNN
+F 3 "" H 1600 5400 50  0001 C CNN
+	1    1600 5400
+	1    0    0    -1
+$EndComp
+Wire Wire Line
+	1500 5400 1500 5300
+Connection ~ 1500 5400
+Wire Wire Line
+	1600 5400 1500 5400
+$Comp
+L power:+12V #PWR0111
+U 1 1 61774C31
+P 2850 5350
+F 0 "#PWR0111" H 2850 5200 50  0001 C CNN
+F 1 "+12V" H 2850 5500 50  0000 C CNN
+F 2 "" H 2850 5350 50  0001 C CNN
+F 3 "" H 2850 5350 50  0001 C CNN
+	1    2850 5350
+	1    0    0    -1
+$EndComp
+Wire Wire Line
+	2850 5350 2750 5350
+Wire Wire Line
+	2750 5250 2750 5350
+Connection ~ 2750 5350
+$Comp
+L power:-12V #PWR0112
+U 1 1 6177FFC5
+P 4050 5400
+F 0 "#PWR0112" H 4050 5500 50  0001 C CNN
+F 1 "-12V" H 4050 5550 50  0000 C CNN
+F 2 "" H 4050 5400 50  0001 C CNN
+F 3 "" H 4050 5400 50  0001 C CNN
+	1    4050 5400
+	-1   0    0    1
+$EndComp
+Wire Wire Line
+	2100 6400 2900 6400
+Wire Wire Line
+	2900 6400 3700 6400
 Wire Bus Line
 	4350 3700 4350 5200
