File: SE-030.kicad_pcb (KiCad board)
At the start: 4 copper layers, 195.2 x 99.6 mm, 100 parts, among them J1 MacSEPDS, SW1 OSCSEL, U1 XC95144XL-TQ100, U10 39SF040, U11 39SF040, U13 74AHCT573, U14 MC68HC000FN20, U15 74AHCT573, U16 74AHCT573, U17 74AHCT573, U18 74AHCT573, U19 74AHCT573, U2 74AHCT573, U20 74AHCT573, U21 74AHCT573, U22 74AHCT573, U23 74AHCT573, U24 74AHCT573, U4 20M, U5 25M, U8 KM48C2100, U9 KM48C2100

Commit message: more
Parts:
- moved C5 14.1 mm to (118.0, 77.2)
- moved C6 14.1 mm to (122.0, 77.2)
- moved R1 14.1 mm to (120.7, 85.3)
- moved R10 14.1 mm to (116.3, 77.2)
- moved R11 14.1 mm to (120.3, 77.2)
- moved R2 14.1 mm to (119.2, 85.3)
- moved U4 14.1 mm to (121.1, 81.0)
- moved U5 14.1 mm to (117.1, 81.0)
- moved C33 3.50 mm to (124.8, 118.8)
- moved C34 3.50 mm to (109.6, 107.3)
- moved C35 3.50 mm to (118.2, 118.8)
- moved C36 3.50 mm to (118.5, 99.5)
- moved C41 3.50 mm to (126.0, 99.5)
- moved C43 3.50 mm to (128.9, 113.8)
- moved C44 3.50 mm to (109.6, 102.3)
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Routing:
- net /Buf/AccD14: track 97.6 -> 128.7 mm
- net /Buf/AccD11: track 100.4 -> 131.3 mm
- net /Buf/AccD15: track 102.0 -> 132.5 mm
- net /Buf/AccD10: track 101.8 -> 131.5 mm
- net /Buf/AccD9: track 100.7 -> 128.9 mm
- net /Buf/AccD7: track 124.1 -> 152.2 mm
- net /Buf/AccD6: track 123.6 -> 151.6 mm
- net /Buf/AccD8: track 95.4 -> 122.8 mm
- net /Buf/AccD5: track 130.2 -> 156.4 mm
- net /Buf/AccD4: track 136.4 -> 155.0 mm
- net /Buf/AccD3: track 131.8 -> 149.6 mm
- net /Buf/AccD2: track 127.2 -> 143.1 mm
- net /Buf/AccD1: track 126.3 -> 140.1 mm
- net +3V3: track 48.1 -> 35.0 mm, vias 40 -> 10
- net /Buf/AccD0: track 120.7 -> 132.9 mm
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- added copper zone on F.Cu, net +3V3

Commit message: Add LC... sloppy
Parts:
- removed the C1 at (125.1, 53.6)
- removed the C1 at (146.7, 53.6)
- removed the C1 at (172.1, 53.6)
- removed the C1 at (150.5, 53.6)
- removed the C1 at (149.4, 75.8)
- removed the C1 at (124.0, 75.8)
- removed C11: 2u2, stdpads:C_0603
- removed the C18 at (68.8, 91.2)
- removed the C2 at (102.6, 73.2)
- removed C21, C23, C25: 10u, stdpads:C_0805
- removed the C26 at (98.8, 63.9)
- removed the C27 at (98.8, 66.3)
- removed the C28 at (102.6, 63.9)
- removed the C29 at (98.8, 68.8)
- removed the C30 at (102.6, 66.3)
- removed the C31 at (106.5, 63.9)
- removed the C32 at (102.6, 68.8)
- removed the C37 at (72.1, 77.7)
- removed the C38 at (72.1, 80.2)
- removed the C39 at (76.0, 77.7)
- removed the C40 at (72.1, 82.6)
- removed the C41 at (76.0, 80.2)
- removed the C42 at (79.8, 77.7)
- removed R12, R6: 22, stdpads:R_0603
- added C8: 10u, stdpads:C_0805, F.Cu at (118.1, 91.8)
- added C9: 10u, stdpads:C_0805, F.Cu at (115.8, 76.3)
- added J2: JTAG, Connector:Tag-Connect_TC2070-IDC-FP_2x07_P1.27mm_Vertical, F.Cu at (113.0, 49.7)
- added U3: AZ1117CH-3.3, stdpads:SOT-223, F.Cu at (115.0, 87.6)
- added U6: AZ1117CH2-3.3, stdpads:SOT-223, F.Cu at (118.6, 66.8)
- C10, C7: value 2u2 -> 10u; footprint stdpads:C_0603 -> stdpads:C_0805
- C12, C13, C14, C15, C16, C17: footprint stdpads:C_0603 -> stdpads:C_0805
- U10, U11: footprint stdpads:PLCC-32_SMDSocket -> stdpads:PLCC-32
- U14: footprint Package_LCC:PLCC-68_SMD-Socket -> stdpads:PLCC-68
- moved FID2 158.0 mm to (210.3, 45.0)
- moved H2 149.3 mm to (210.3, 42.4)
- moved FID3 145.3 mm to (210.3, 135.4)
- moved H3 142.2 mm to (210.3, 137.9)
- moved C20 131.8 mm to (195.5, 51.6), turned to 270 degrees
- moved C24 131.6 mm to (197.9, 51.6), turned to 270 degrees
- moved H4 129.5 mm to (196.5, 137.9)
- moved C19 128.8 mm to (197.9, 121.1), turned to 90 degrees
- moved C22 126.1 mm to (193.0, 51.6), turned to 270 degrees
- moved C15 120.1 mm to (172.1, 55.8), turned to 270 degrees
- moved C14 100.4 mm to (150.5, 55.8), turned to 270 degrees
- moved C13 91.0 mm to (146.7, 55.8), turned to 270 degrees
- moved C17 87.4 mm to (149.4, 75.8), turned to 270 degrees
- moved C12 76.8 mm to (125.1, 55.8), turned to 270 degrees
- moved SW1 76.0 mm to (107.3, 123.2), turned to 180 degrees
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- renumbered C1 to C18, C1 to C2, C36 to C26, C41 to C27, C43 to C28, C33 to C29, C35 to C30, C34 to C31, C44 to C32, C14 to C33, C14 to C34, C14 to C35, C14 to C36, C14 to C37, C14 to C38, C14 to C39, C14 to C40, C14 to C41, C14 to C42, C14 to C43, C14 to C44, R10 to R3, R11 to R4
Connections:
- C10 pad 1: +5V -> +3V3
- J1 pad A31: Net-(J1-PadA31) -> +12V
- J1 pad A32: Net-(J1-PadA32) -> +12V
- J1 pad B30: Net-(J1-PadB30) -> +12V
- J1 pad B31: Net-(J1-PadB31) -> +12V
- J1 pad B32: Net-(J1-PadB32) -> -5V
- J1 pad C12: /MC68k/~HALT~ -> /Control/~RESET~
- J1 pad C32: Net-(J1-PadC32) -> -12V
- R3 pad 1: GND -> +3V3
- R3 pad 2: Net-(R10-Pad2) -> /Control/SW1
- R4 pad 1: GND -> +3V3
- R4 pad 2: Net-(R11-Pad2) -> /Clk.sch/CK20EN
- SW1 pad 1: Net-(R11-Pad2) -> /Clk.sch/CK20EN
- SW1 pad 2: Net-(R10-Pad2) -> /Control/SW1
- SW1 pad 3: Net-(R12-Pad2) -> GND
- SW1 pad 4: Net-(R12-Pad2) -> GND
- U1 pad 10: /MC68k/~HALT~ -> /Control/A12
- U1 pad 11: /Control/A23 -> /Control/A13
- U1 pad 12: /Control/A22 -> /Control/A14
- U1 pad 13: /Control/A21 -> /Control/A15
- U1 pad 14: /Control/A20 -> /Control/A16
- U1 pad 15: /Control/A19 -> /Control/A17
- U1 pad 17: /Control/A17 -> /Control/A19
- U1 pad 18: /Control/A16 -> /Control/A20
- U1 pad 19: /Control/A15 -> /Control/A21
- U1 pad 2: /Buf/Aout~OE~ -> /Control/A5
- U1 pad 20: /Control/A14 -> /Control/A22
- U1 pad 22: /Control/FCLK -> /Control/C16M
- U1 pad 23: /Control/C16M -> /Control/C8M
- U1 pad 24: Net-(U1-Pad24) -> /Control/A23
- U1 pad 25: Net-(U1-Pad25) -> /PDS/E
- U1 pad 27: /Control/C8M -> /Control/FCLK
- U1 pad 28: Net-(U1-Pad28) -> /Control/Acc~DTACK
- U1 pad 29: Net-(U1-Pad29) -> /Control/AccR~W~
- U1 pad 3: /Buf/ADoutLE1 -> /Control/A6
- U1 pad 30: Net-(U1-Pad30) -> /Control/Acc~LDS~
- U1 pad 32: Net-(U1-Pad32) -> /Control/Acc~AS~
- U1 pad 33: Net-(U1-Pad33) -> /Control/Acc~UDS~
- U1 pad 34: Net-(U1-Pad34) -> /Control/ROM~WE~
- U1 pad 35: /Control/A13 -> /Control/ROM~CS~
- U1 pad 36: /Control/A12 -> /Control/~CAS~
- U1 pad 37: /Control/A11 -> /Control/~OE~
- U1 pad 39: /Control/A10 -> Net-(U1-Pad39)
- U1 pad 4: /Buf/ADoutLE0 -> /Control/A7
- U1 pad 40: /Control/A9 -> /Control/RA4
- U1 pad 41: /Control/A8 -> /Control/RA3
- U1 pad 42: /Control/A7 -> /Control/RA5
- U1 pad 43: /Control/A6 -> /Control/RA2
- U1 pad 45: Net-(U1-Pad45) -> /Control/TDI
- U1 pad 46: /Control/A5 -> /Control/RA6
- U1 pad 47: Net-(U1-Pad47) -> /Control/TMS
- U1 pad 48: Net-(U1-Pad48) -> /Control/TCK
- U1 pad 49: /Control/A4 -> Net-(U1-Pad49)
- U1 pad 50: /Control/RA4 -> /Control/RA1
- U1 pad 52: /Control/RA5 -> /Control/RA7
- U1 pad 53: /Control/RA6 -> /Control/RA0
- U1 pad 54: /Control/RA7 -> /Control/RA8
- U1 pad 55: /Control/RA8 -> /Control/RA10
- U1 pad 58: /Control/RA10 -> Net-(U1-Pad58)
- U1 pad 59: /Control/RA11 -> /Clk.sch/CK25EN
- U1 pad 6: /Buf/Dout~OE~ -> /Control/A8
- U1 pad 60: /Control/~RAS~ -> /Control/SW1
- U1 pad 61: /Control/~CAS~ -> Net-(U1-Pad61)
- U1 pad 63: /Control/ROM~CS~ -> /Control/RA11
- U1 pad 64: /Control/~OE~ -> /Control/~RAS~
- U1 pad 67: /Control/Acc~UDS~ -> /Clk.sch/CK20EN
- U1 pad 68: /Control/Acc~LDS~ -> Net-(U1-Pad68)
- U1 pad 7: /Buf/Din~OE~ -> /Control/A9
- U1 pad 70: /Control/Acc~AS~ -> Net-(U1-Pad70)
- U1 pad 71: /Control/Acc~DTACK -> Net-(U1-Pad71)
- U1 pad 72: /Control/Acc~BERR~ -> Net-(U1-Pad72)
- U1 pad 73: /Control/Acc~VPA~ -> Net-(U1-Pad73)
- U1 pad 74: /Control/A3 -> /Control/Mac~VMA~
- U1 pad 76: /Control/A2 -> /Control/Mac~BERR~
- U1 pad 77: /Control/A1 -> /Control/Mac~VPA~
- U1 pad 78: /Control/AccR~W~ -> /Control/Mac~DTACK~
- U1 pad 79: Net-(U1-Pad79) -> /Control/Mac~LDS~
- U1 pad 8: /Buf/DinLE -> /Control/A10
- U1 pad 80: Net-(U1-Pad80) -> /Control/Mac~UDS~
- U1 pad 81: /Control/RA0 -> /Control/Mac~AS~
- U1 pad 82: /Control/RA1 -> /Buf/ADoutLE1
- U1 pad 83: Net-(U1-Pad83) -> /Control/TDO
- U1 pad 85: /Control/RA2 -> /Buf/ADoutLE0
- U1 pad 86: /Control/RA3 -> /Buf/DinLE
- U1 pad 87: /Control/Mac~AS~ -> /Buf/Aout~OE~
- U1 pad 89: /Control/Mac~VMA~ -> /Buf/Dout~OE~
- U1 pad 9: /Control/~WAIT~ -> /Control/A11
- U1 pad 90: /Control/Mac~LDS~ -> /Buf/Din~OE~
- U1 pad 91: /Control/Mac~UDS~ -> /Control/~RESET~
- U1 pad 92: /Control/Mac~DTACK~ -> /Control/Acc~BERR~
- U1 pad 93: /Control/Mac~VPA~ -> /Control/Acc~VPA~
- U1 pad 94: /Control/Mac~BERR~ -> /Control/A1
- U1 pad 95: /PDS/E -> /Control/A2
- U1 pad 96: Net-(U1-Pad96) -> /Control/A3
- U1 pad 97: Net-(U1-Pad97) -> /Control/A4
- U10 pad 1: /Control/A19 -> /Control/A15
- U10 pad 10: /Control/A3 -> /Control/A5
- U10 pad 11: /Control/A2 -> /Control/A6
- U10 pad 12: /Control/A1 -> /Control/A7
- U10 pad 2: /Control/A17 -> /Control/A9
- U10 pad 23: /Control/A11 -> /Control/A12
- U10 pad 25: /Control/A12 -> /Control/A13
- U10 pad 26: /Control/A10 -> /Control/A16
- U10 pad 27: /Control/A9 -> /Control/A17
- U10 pad 28: /Control/A14 -> /Control/A18
- U10 pad 29: /Control/A15 -> /Control/A19
- U10 pad 3: /Control/A16 -> /Control/A14
- U10 pad 30: /Control/A18 -> /Control/A8
- U10 pad 31: /Control/L~WE~ -> /Control/ROM~WE~
- U10 pad 32: +3V3 -> +5V
- U10 pad 4: /Control/A13 -> /Control/A11
- U10 pad 5: /Control/A8 -> /Control/A10
- U10 pad 6: /Control/A7 -> /Control/A1
- U10 pad 7: /Control/A6 -> /Control/A2
- U10 pad 8: /Control/A5 -> /Control/A3
- U11 pad 1: /Control/A19 -> /Control/A9
- U11 pad 10: /Control/A3 -> /Control/A11
- U11 pad 11: /Control/A2 -> /Control/A14
- U11 pad 12: /Control/A1 -> /Control/A15
- U11 pad 2: /Control/A17 -> /Control/A1
- U11 pad 23: /Control/A11 -> /Control/A8
- U11 pad 25: /Control/A12 -> /Control/A19
- U11 pad 26: /Control/A10 -> /Control/A18
- U11 pad 27: /Control/A9 -> /Control/A17
- U11 pad 28: /Control/A14 -> /Control/A16
- U11 pad 29: /Control/A15 -> /Control/A13
- U11 pad 3: /Control/A16 -> /Control/A3
- U11 pad 30: /Control/A18 -> /Control/A12
- U11 pad 31: /Control/U~WE~ -> /Control/ROM~WE~
- U11 pad 32: +3V3 -> +5V
- U11 pad 4: /Control/A13 -> /Control/A7
- U11 pad 5: /Control/A8 -> /Control/A6
- U11 pad 6: /Control/A7 -> /Control/A5
- U11 pad 7: /Control/A6 -> /Control/A4
- U11 pad 8: /Control/A5 -> /Control/A2
- U11 pad 9: /Control/A4 -> /Control/A10
- U14 pad 19: /MC68k/~HALT~ -> /Control/~RESET~
- U14 pad 20: /MC68k/~HALT~ -> /Control/~RESET~
- U4 pad 1: Net-(R11-Pad2) -> /Clk.sch/CK20EN
- U5 pad 1: Net-(R10-Pad2) -> /Clk.sch/CK25EN
- U8 pad 1: VDD -> +5V
- U8 pad 14: VDD -> +5V
- U8 pad 2: /Buf/AccD0 -> /Buf/AccD7
- U8 pad 24: /Buf/AccD4 -> /Buf/AccD0
- U8 pad 25: /Buf/AccD5 -> /Buf/AccD2
- U8 pad 26: /Buf/AccD6 -> /Buf/AccD4
- U8 pad 27: /Buf/AccD7 -> /Buf/AccD6
- U8 pad 3: /Buf/AccD1 -> /Buf/AccD5
- U8 pad 4: /Buf/AccD2 -> /Buf/AccD3
- U8 pad 5: /Buf/AccD3 -> /Buf/AccD1
- U9 pad 1: VDD -> +5V
- U9 pad 10: /Control/RA0 -> /Control/RA1
- U9 pad 11: /Control/RA1 -> /Control/RA0
- U9 pad 12: /Control/RA2 -> /Control/RA10
- U9 pad 13: /Control/RA3 -> /Control/RA11
- U9 pad 14: VDD -> +5V
- U9 pad 16: /Control/RA4 -> /Control/RA9
- U9 pad 17: /Control/RA5 -> /Control/RA8
- U9 pad 18: /Control/RA6 -> /Control/RA7
- U9 pad 19: /Control/RA7 -> /Control/RA6
- U9 pad 2: /Buf/AccD8 -> /Buf/AccD15
- U9 pad 20: /Control/RA8 -> /Control/RA5
- U9 pad 21: /Control/RA9 -> /Control/RA4
- U9 pad 24: /Buf/AccD12 -> /Buf/AccD8
- U9 pad 25: /Buf/AccD13 -> /Buf/AccD10
- U9 pad 26: /Buf/AccD14 -> /Buf/AccD12
- U9 pad 27: /Buf/AccD15 -> /Buf/AccD14
- U9 pad 3: /Buf/AccD9 -> /Buf/AccD13
- U9 pad 4: /Buf/AccD10 -> /Buf/AccD11
- U9 pad 5: /Buf/AccD11 -> /Buf/AccD9
- U9 pad 8: /Control/RA11 -> /Control/RA3
- U9 pad 9: /Control/RA10 -> /Control/RA2
Routing:
- net +3V3: track 35.0 -> 179.2 mm, vias 10 -> 13
- net /Control/~RESET~: track 0.00 -> 123.7 mm, vias 0 -> 4
- net /Control/TDO: track 0.00 -> 109.2 mm, vias 0 -> 2
- net /MC68k/~HALT~: track 98.3 -> 0.00 mm, vias 4 -> 0
- net /Control/U~WE~: track 29.5 -> 124.2 mm, vias 3 -> 2
- net /Control/A8: track 72.3 -> 158.2 mm, vias 2 -> 4
- net /Control/A17: track 53.9 -> 136.6 mm, vias 2 -> 4
- net /Control/ROM~CS~: track 2.01 -> 83.9 mm, vias 1 -> 3
- net /Control/~OE~: track 62.2 -> 141.4 mm
- net /Control/A16: track 64.2 -> 139.5 mm, vias 2 -> 4
- net /Control/L~WE~: track 20.9 -> 94.8 mm, vias 1 -> 0
- net /Control/~RAS~: track 53.7 -> 125.5 mm, vias 3 -> 2
- net /Control/RA3: track 43.9 -> 115.6 mm, vias 3 -> 4
- net /Control/RA4: track 42.6 -> 113.2 mm, vias 2 -> 4
- net /Control/TDI: track 0.00 -> 70.1 mm, vias 0 -> 2
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- added copper zone on In2.Cu, net +5V
- added copper zone on In1.Cu, net GND
Other:
- board size 195.2 x 99.6 mm -> 109.1 x 99.6 mm
- board text added: "20 MHz"
- board text added: "25 MHz"
- board text added: "4406A"
- board text added: "Accelerator for Mac SE"
- board text added: "Clock Select"
- board text added: "GW"
- board text added: "Garrett’s Workshop"
- board text added: "Warp-SE"
