File: SE30/Control.sch (KiCad schematic (older format))
At the start: 8 parts, among them U1 XC95144XL-TQ100

Commit message: Add LC... sloppy
Connections:
- net Acc~AS~: now also U1.33 (P33); no longer U1.32 (P32)
- net Acc~UDS~: now also U1.32 (P32); no longer U1.33 (P33)
- net Mac~BERR~: now also U1.74 (P74); no longer U1.76 (P76)
- net Mac~VMA~: now also U1.77 (P77); no longer U1.74 (P74)
- net Mac~VPA~: now also U1.76 (P76); no longer U1.77 (P77)
- net CKEN: no longer names the net of U1.59 (P59)
- net SW0: no longer names the net of U1.67 (P67)
- net SW1: no longer names the net of U1.60 (P60)
- net TCK: no longer names the net of U1.48 (TCK)
- net TDI: no longer names the net of U1.45 (TDI)
- net TDO: no longer names the net of U1.83 (TDO)
- net TMS: no longer names the net of U1.47 (TMS)
Changed lines of the file:
@@
 $Descr A4 11693 8268
 encoding utf-8
-Sheet 7 10
+Sheet 8 10
 Title ""
 Date ""
@@
 Text HLabel 10400 2900 2    50   Output ~ 0
 Mac~AS~
-Text HLabel 10400 2300 2    50   Output ~ 0
+Text HLabel 10400 2500 2    50   Output ~ 0
 Mac~VMA~
 Text HLabel 10400 2600 2    50   Input ~ 0
 Mac~DTACK~
-Text HLabel 10400 2500 2    50   Input ~ 0
+Text HLabel 10400 2400 2    50   Input ~ 0
 Mac~VPA~
-Text HLabel 10400 2400 2    50   Input ~ 0
+Text HLabel 10400 2300 2    50   Input ~ 0
 Mac~BERR~
 Text HLabel 8400 3600 0    50   Input ~ 0
@@
 Text HLabel 8400 5000 0    50   Output ~ 0
 Acc~VPA~
-Text HLabel 8400 4100 0    50   Input ~ 0
+Text HLabel 8400 4200 0    50   Input ~ 0
 Acc~AS~
 Text HLabel 8400 4000 0    50   Input ~ 0
 Acc~LDS~
-Text HLabel 8400 4200 0    50   Input ~ 0
+Text HLabel 8400 4100 0    50   Input ~ 0
 Acc~UDS~
 Text HLabel 8400 4900 0    50   Output ~ 0
@@
 Entry Wire Line
 	10700 1400 10600 1500
-Text HLabel 10400 4900 2    50   Input ~ 0
-SW0
-Text HLabel 10400 4200 2    50   Input ~ 0
-SW1
-Text HLabel 10400 4100 2    50   Output ~ 0
-CKEN
-Text HLabel 10400 5600 2    50   Input ~ 0
-TDI
-Text HLabel 10400 5700 2    50   Input ~ 0
-TMS
-Text HLabel 10400 5800 2    50   Input ~ 0
-TCK
-Text HLabel 10400 5900 2    50   Output ~ 0
-TDO
 Wire Bus Line
 	10700 1400 10700 1800
