File: SE30/RAMROM.sch (KiCad schematic (older format))
At the start: 10 parts, among them U10 39SF040, U11 39SF040, U8 KM48C2100, U9 KM48C2100

Commit message: Add LC... sloppy
Parts:
- C12, C13, C14, C15, C16, C17: footprint stdpads:C_0805 -> stdpads:C_0603
- U10, U11: footprint stdpads:PLCC-32 -> stdpads:PLCC-32_SMDSocket
Connections:
- net labels added: +3V3, VMEM
- net labels removed: ROM~WE~
